Commit message: Update URDF and Inverse Kinematics

File: host_serial_control/moveo.URDF (robot description, URDF)
Before this commit: robot moveo_urdf_5, 12 links, 11 joints
Links:
- removed link Gripper_Idol_Gear
- removed link Gripper_Servo_Gear
- removed link Pivot_Arm_Gripper_Idol
- removed link Pivot_Arm_Gripper_Servo
- removed link Tip_Gripper_Idol
- removed link Tip_Gripper_Servo
- link Link_1: geometry 
- link Link_2: geometry 
- link Link_3: geometry 
- link Link_4: geometry collision mesh filename=package://moveo_urdf_5/meshes/Link_4.STL
- link Link_5: geometry 
- link base_link: geometry 
Joints:
- removed joint Gripper_Idol_Gear_Joint
- removed joint Gripper_Servo_Gear_Joint
- removed joint Pivot_Arm_Gripper_Idol_Joint
- removed joint Pivot_Arm_Gripper_Servo_Joint
- removed joint Tip_Gripper_Idol_Joint
- removed joint Tip_Gripper_Servo_Joint
